File: PCB/totem_0-3/totem_0_3.kicad_pcb (KiCad board)
At the start: 2 copper layers, 130.7 x 94.4 mm, 29 parts, among them SW1 SW_Push_45deg, SW10 SW_Push_45deg, SW11 SW_Push_45deg, SW12 SW_Push_45deg, SW13 SW_Push_45deg, SW14 SW_Push_45deg, SW15 SW_Push_45deg, SW16 SW_Push_45deg, SW17 SW_Push_45deg, SW18 SW_Push_45deg, SW19 SW_Push_45deg, SW2 SW_Push_45deg, SW3 SW_Push_45deg, SW4 SW_Push_45deg, SW5 SW_Push_45deg, SW6 SW_Push_45deg, SW7 SW_Push_45deg, SW8 SW_Push_45deg, SW9 SW_Push_45deg, U3 nice_nano

Commit message: n!n version
Parts:
- removed BAT+1: +, TOTEMlib:BatteryPad
- removed BATGND1: -, TOTEMlib:BatteryPad
- removed REF** (x4): MountingHole_3.2mm_M3_DIN965_Pad, MountingHole:MountingHole_3.2mm_M3_DIN965_Pad
- removed SW1, SW10, SW11, SW12, SW13, SW14, SW15, SW16, SW17, SW18, SW19, SW2, SW3, SW4, SW5, SW6, SW7, SW8, SW9: SW_Push_45deg, switches:Kailh_socket_PG1350_reversible
- removed U3: nice_nano, nice-nano:nice_nano
- added D1: 1N4148W, Diode_SMD:D_SOD-123_Reversible_THT, F.Cu at (68.9, 94.2)
- added D10: 1N4148W, Diode_SMD:D_SOD-123_Reversible_THT, F.Cu at (124.3, 81.4)
- added D11: 1N4148W, Diode_SMD:D_SOD-123_Reversible_THT, F.Cu at (124.3, 64.4)
- added D12: 1N4148W, Diode_SMD:D_SOD-123_Reversible_THT, F.Cu at (124.3, 47.4)
- added D13: 1N4148W, Diode_SMD:D_SOD-123_Reversible_THT, F.Cu at (142.4, 84.4)
- added D14: 1N4148W, Diode_SMD:D_SOD-123_Reversible_THT, F.Cu at (142.7, 67.4)
- added D15: 1N4148W, Diode_SMD:D_SOD-123_Reversible_THT, F.Cu at (143.0, 50.4)
- added D16: 1N4148W, Diode_SMD:D_SOD-123_Reversible_THT, F.Cu at (160.5, 89.7)
- added D17: 1N4148W, Diode_SMD:D_SOD-123_Reversible_THT, F.Cu at (161.1, 72.7)
- added D18: 1N4148W, Diode_SMD:D_SOD-123_Reversible_THT, F.Cu at (161.7, 55.7)
- added D19: 1N4148W, Diode_SMD:D_SOD-123_Reversible_THT, F.Cu at (146.7, 108.4)
- added D2: 1N4148W, Diode_SMD:D_SOD-123_Reversible_THT, F.Cu at (67.5, 77.3)
- added D20: 1N4148W, Diode_SMD:D_SOD-123_Reversible_THT, F.Cu at (165.6, 112.9)
- added D21: 1N4148W, Diode_SMD:D_SOD-123_Reversible_THT, F.Cu at (180.4, 125.3)
- added D22: 1N4148W, Diode_SMD:D_SOD-123_Reversible_THT, B.Cu at (188.6, 83.9)
- added D3: 1N4148W, Diode_SMD:D_SOD-123_Reversible_THT, F.Cu at (66.0, 60.4)
- added D4: 1N4148W, Diode_SMD:D_SOD-123_Reversible_THT, F.Cu at (86.9, 92.7)
- added D5: 1N4148W, Diode_SMD:D_SOD-123_Reversible_THT, F.Cu at (85.4, 75.7)
- added D6: 1N4148W, Diode_SMD:D_SOD-123_Reversible_THT, F.Cu at (83.9, 58.8)
- added D7: 1N4148W, Diode_SMD:D_SOD-123_Reversible_THT, F.Cu at (104.9, 83.4)
- added D8: 1N4148W, Diode_SMD:D_SOD-123_Reversible_THT, F.Cu at (104.0, 66.4)
- added D9: 1N4148W, Diode_SMD:D_SOD-123_Reversible_THT, F.Cu at (103.1, 49.4)
- added H1: MountingHole, TOTEMlib:M2-sandwich-hole, F.Cu at (193.2, 102.3)
- added H2: MountingHole, TOTEMlib:M2-sandwich-hole, F.Cu at (76.8, 80.3)
- added H4: MountingHole, TOTEMlib:M2-sandwich-hole, F.Cu at (113.7, 45.0)
- added H5: MountingHole, TOTEMlib:M2-sandwich-hole, F.Cu at (197.5, 40.7)
- added H6: MountingHole, TOTEMlib:M2-sandwich-hole, F.Cu at (132.8, 85.9)
- added J1: Conn_01x02_Socket, Connector_JST:JST_PH_S2B-PH-K_1x02_P2.00mm_Horizontal, F.Cu at (191.2, 75.2)
- added RSW2: SW_Push, Button_Switch_SMD:SW_SPST_B3U-1000P, B.Cu at (178.3, 76.3)
- added S1: SW_Push_45deg, keyswitches:wubbo-choc-socket-reversible, F.Cu at (68.6, 89.6)
- added S10: SW_Push_45deg, keyswitches:wubbo-choc-socket-reversible, F.Cu at (124.4, 76.7)
- added S11: SW_Push_45deg, keyswitches:wubbo-choc-socket-reversible, F.Cu at (124.4, 59.7)
- added S12: SW_Push_45deg, keyswitches:wubbo-choc-socket-reversible, F.Cu at (124.4, 42.7)
- added S13: SW_Push_45deg, keyswitches:wubbo-choc-socket-reversible, F.Cu at (142.6, 79.7)
- added S14: SW_Push_45deg, keyswitches:wubbo-choc-socket-reversible, F.Cu at (142.8, 62.7)
- added S15: SW_Push_45deg, keyswitches:wubbo-choc-socket-reversible, F.Cu at (143.1, 45.7)
- added S16: SW_Push_45deg, keyswitches:wubbo-choc-socket-reversible, F.Cu at (160.7, 85.0)
- added S17: SW_Push_45deg, keyswitches:wubbo-choc-socket-reversible, F.Cu at (161.3, 68.0)
- added S18: SW_Push_45deg, keyswitches:wubbo-choc-socket-reversible, F.Cu at (161.9, 51.0)
- added S19: SW_Push_45deg, keyswitches:wubbo-choc-socket-reversible, F.Cu at (146.9, 103.8)
- added S2: SW_Push_45deg, keyswitches:wubbo-choc-socket-reversible, F.Cu at (67.1, 72.6)
- added S20: SW_Push_45deg, keyswitches:wubbo-choc-socket-reversible, F.Cu at (167.7, 108.8)
- added S21: SW_Push_45deg, keyswitches:wubbo-choc-socket-reversible, F.Cu at (183.8, 116.7)
- added S3: SW_Push_45deg, keyswitches:wubbo-choc-socket-reversible, F.Cu at (65.6, 55.7)
- added S4: SW_Push_45deg, keyswitches:wubbo-choc-socket-reversible, F.Cu at (86.5, 88.0)
- added S5: SW_Push_45deg, keyswitches:wubbo-choc-socket-reversible, F.Cu at (85.0, 71.1)
- added S6: SW_Push_45deg, keyswitches:wubbo-choc-socket-reversible, F.Cu at (83.6, 54.1)
- added S7: SW_Push_45deg, keyswitches:wubbo-choc-socket-reversible, F.Cu at (104.7, 78.7)
- added S8: SW_Push_45deg, keyswitches:wubbo-choc-socket-reversible, F.Cu at (103.8, 61.8)
- added S9: SW_Push_45deg, keyswitches:wubbo-choc-socket-reversible, F.Cu at (102.9, 44.8)
- added SW22: RotaryEncoder_Switch, Keebio-Parts:RotaryEncoder_Alps_EC11E-Switch_Vertical_H20mm, F.Cu at (183.3, 89.0)
- added U1: nice_nano, keyboard-reversible:ProMicro_unrouted_MAC8, F.Cu at (183.7, 55.8)
- PSW1, PSW2: value SW_SPDT -> SW_Push_SPDT; footprint TOTEMlib:MSK12C02 -> kleeb-master-switches:switch-MSK-12C02-smd
- RSW1: footprint kbd:ResetSW -> Button_Switch_SMD:SW_SPST_B3U-1000P
- moved PSW2 252.3 mm to (183.9, 38.0)
- moved PSW1 252.3 mm to (183.9, 38.0), turned to -90 degrees
- moved RSW1 161.7 mm to (178.3, 76.3), turned to -90 degrees
Connections:
- net BAT+_L renamed VBAT
- PSW1 pad 3: VBAT_L -> BAT+
- PSW2 pad 1: unconnected-(PSW2-A-Pad1) -> BAT+
- PSW2 pad 3: VBAT_L -> unconnected-(PSW2-C-Pad3)
- RSW1 pad 1: RESET_L -> RESET
- RSW1 pad 2: GND_L -> GND
Routing:
- net /C1: track 0.00 -> 219.6 mm, vias 0 -> 5
- net /C4: track 0.00 -> 207.2 mm, vias 0 -> 9
- net /C2: track 0.00 -> 192.5 mm, vias 0 -> 4
- net /S1: track 177.3 -> 0.00 mm, vias 1 -> 0
- net /S16: track 167.0 -> 0.00 mm, vias 1 -> 0
- net /C3: track 0.00 -> 165.5 mm, vias 0 -> 4
- net /S2: track 164.2 -> 0.00 mm, vias 1 -> 0
- net /C5: track 0.00 -> 163.5 mm, vias 0 -> 6
- net /S6: track 158.5 -> 0.00 mm, vias 1 -> 0
- net /C6: track 0.00 -> 155.2 mm, vias 0 -> 6
- net /S7: track 152.3 -> 0.00 mm, vias 1 -> 0
- net R1: track 0.00 -> 146.8 mm, vias 0 -> 2
- net /S11: track 143.5 -> 0.00 mm, vias 1 -> 0
- net /S12: track 143.3 -> 0.00 mm, vias 1 -> 0
- net R3: track 0.00 -> 131.4 mm, vias 0 -> 1
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- added copper zone on B.Cu, net GND
- added copper zone on F.Cu, net GND
- removed copper zone on B.Cu, net GND_L
- removed copper zone on F.Cu, net GND_L
Other:
- board size 130.7 x 94.4 mm -> 146.7 x 102.8 mm
- board text added: "MCU Face up. Solder jumpers on other side."
- board text removed: "0.1"
- board text removed: "A N O T T H A T"
- board text removed: "BT+"
- board text removed: "BT-"
- board text removed: "C0"
- board text removed: "C1"
- board text removed: "C2"
- board text removed: "C3"
- board text removed: "C4"
- board text removed: "GND"
- board text removed: "M A D E B Y"
- board text removed: "R E V I S I O N 0 . 3"
- board text removed: "R0"
- board text removed: "R1"
- board text removed: "R2"
- board text removed: "R3"
- board text removed: "RST"
- board text removed: "RX"
- board text removed: "S C A R Y G E I S T"
- board text removed: "T O T E M"
- board text removed: "TX"
- board text removed: "VCC"
