File: PCB/totem_0-3/totem_0_3.kicad_sch (KiCad schematic)
At the start: 25 parts, among them SW1 SW_Push_45deg, SW10 SW_Push_45deg, SW11 SW_Push_45deg, SW12 SW_Push_45deg, SW13 SW_Push_45deg, SW14 SW_Push_45deg, SW15 SW_Push_45deg, SW16 SW_Push_45deg, SW17 SW_Push_45deg, SW18 SW_Push_45deg, SW19 SW_Push_45deg, SW2 SW_Push_45deg, SW3 SW_Push_45deg, SW4 SW_Push_45deg, SW5 SW_Push_45deg, SW6 SW_Push_45deg, SW7 SW_Push_45deg, SW8 SW_Push_45deg, SW9 SW_Push_45deg, U3 nice_nano

Commit message: n!n version
Parts:
- removed BAT+1: +, TOTEMlib:BatteryPad, symbol Mechanical:MountingHole_Pad
- removed BATGND1: -, TOTEMlib:BatteryPad, symbol Mechanical:MountingHole_Pad
- removed PSW1, PSW2: SW_SPDT, TOTEMlib:MSK12C02, symbol Switch:SW_SPDT
- removed U3: nice_nano, nice-nano:nice_nano, symbol nice-nano:nice_nano
- added D1, D10, D11, D12, D13, D14, D15, D16, D17, D18, D19, D2, D20, D21, D22, D3, D4, D5, D6, D7, D8, D9: 1N4148W, Diode_SMD:D_SOD-123_Reversible_THT, symbol Diode:1N4148W
- added H1, H2, H4, H5, H6: MountingHole, TOTEMlib:M2-sandwich-hole, symbol Mechanical:MountingHole
- added J1: Conn_01x02_Socket, Connector_JST:JST_PH_S2B-PH-K_1x02_P2.00mm_Horizontal, symbol Connector:Conn_01x02_Socket
- added PSW1, PSW2: SW_Push_SPDT, kleeb-master-switches:switch-MSK-12C02-smd, symbol Switch:SW_Push_SPDT
- added RSW2: SW_Push, Button_Switch_SMD:SW_SPST_B3U-1000P, symbol Switch:SW_Push
- added S2, S3: SW_Push_45deg, keyswitches:wubbo-choc-socket-reversible, symbol Switch:SW_Push_45deg
- added SW22: RotaryEncoder_Switch, Keebio-Parts:RotaryEncoder_Alps_EC11E-Switch_Vertical_H20mm, symbol Device:RotaryEncoder_Switch
- added U1: nice_nano, keyboard-reversible:ProMicro_unrouted_MAC8, symbol nice-nano:nice_nano
- RSW1: footprint kbd:ResetSW -> Button_Switch_SMD:SW_SPST_B3U-1000P
- S1: renamed from SW16; footprint switches:Kailh_socket_PG1350_reversible -> keyswitches:wubbo-choc-socket-reversible
- S10: renamed from SW3; footprint switches:Kailh_socket_PG1350_reversible -> keyswitches:wubbo-choc-socket-reversible
- S11: renamed from SW8; footprint switches:Kailh_socket_PG1350_reversible -> keyswitches:wubbo-choc-socket-reversible
- S12: renamed from SW13; footprint switches:Kailh_socket_PG1350_reversible -> keyswitches:wubbo-choc-socket-reversible
- S13: renamed from SW4; footprint switches:Kailh_socket_PG1350_reversible -> keyswitches:wubbo-choc-socket-reversible
- S14: renamed from SW9; footprint switches:Kailh_socket_PG1350_reversible -> keyswitches:wubbo-choc-socket-reversible
- S15: renamed from SW14; footprint switches:Kailh_socket_PG1350_reversible -> keyswitches:wubbo-choc-socket-reversible
- S16: renamed from SW5; footprint switches:Kailh_socket_PG1350_reversible -> keyswitches:wubbo-choc-socket-reversible
- S17: renamed from SW10; footprint switches:Kailh_socket_PG1350_reversible -> keyswitches:wubbo-choc-socket-reversible
- S18: renamed from SW15; footprint switches:Kailh_socket_PG1350_reversible -> keyswitches:wubbo-choc-socket-reversible
- S19: renamed from SW17; footprint switches:Kailh_socket_PG1350_reversible -> keyswitches:wubbo-choc-socket-reversible
- S20: renamed from SW18; footprint switches:Kailh_socket_PG1350_reversible -> keyswitches:wubbo-choc-socket-reversible
- S21: renamed from SW19; footprint switches:Kailh_socket_PG1350_reversible -> keyswitches:wubbo-choc-socket-reversible
- S4: renamed from SW1; footprint switches:Kailh_socket_PG1350_reversible -> keyswitches:wubbo-choc-socket-reversible
- S5: renamed from SW6; footprint switches:Kailh_socket_PG1350_reversible -> keyswitches:wubbo-choc-socket-reversible
- S6: renamed from SW11; footprint switches:Kailh_socket_PG1350_reversible -> keyswitches:wubbo-choc-socket-reversible
- S7: renamed from SW2; footprint switches:Kailh_socket_PG1350_reversible -> keyswitches:wubbo-choc-socket-reversible
- S8: renamed from SW7; footprint switches:Kailh_socket_PG1350_reversible -> keyswitches:wubbo-choc-socket-reversible
- S9: renamed from SW12; footprint switches:Kailh_socket_PG1350_reversible -> keyswitches:wubbo-choc-socket-reversible
Connections:
- net S11 is gone; now on net C2: S6.1
- net S15 is gone; now on net C6: S18.1
- net S17 is gone; now on net C4: S19.1
- net S18 is gone; now on net C5: S20.1
- net S19 is gone; now on net C6: S21.1
- net S2 is gone; now on net C3: S7.1
- net S3 is gone; now on net C4: S10.1
- net S4 is gone; now on net C5: S13.1
- net S5 is gone; now on net C6: S16.1
- net S6 is gone; now on net C2: S5.1
- net S7 is gone; now on net C3: S8.1
- net S8 is gone; now on net C4: S11.1
- net S9 is gone; now on net C5: S14.1
- removed net GND_L: RSW1.2, S1.2, S10.2, S11.2, S12.2, S13.2, S14.2, S15.2, S16.2, S17.2, S18.2, S19.2, S20.2, S21.2, S4.2, S5.2, S6.2, S7.2, S8.2, S9.2
- net RESET_L renamed RESET
- net RESET: now also RSW2.2, U1.22 (RST)
- net S1 renamed C2
- net C2: now also U1.5 (P0.17)
- net S10 renamed C6
- net C6: now also SW22.S1, U1.10 (P0.11)
- net S12 renamed C3
- net C3: now also U1.6 (P0.20)
- net S13 renamed C4
- net C4: now also U1.19 (AIN5/P0.29)
- net S14 renamed C5
- net C5: now also U1.8 (P0.24)
- net S16 renamed C1
- net C1: now also S2.1, S3.1, U1.20 (AIN7/P0.31)
- new net: D16.2 (A), S16.2
- new net: D10.2 (A), S10.2
- new net: D13.2 (A), S13.2
- new net: D2.2 (A), S2.2
- new net: D4.2 (A), S4.2
- new net: D15.2 (A), S15.2
- new net: D3.2 (A), S3.2
- new net: D20.2 (A), S20.2
- new net: D8.2 (A), S8.2
- new net: D22.2 (A), SW22.S2
- new net: D18.2 (A), S18.2
- new net: D1.2 (A), S1.2
- new net: D9.2 (A), S9.2
- new net: D19.2 (A), S19.2
- new net: D7.2 (A), S7.2
- new net: D12.2 (A), S12.2
- new net: D6.2 (A), S6.2
- new net: D21.2 (A), S21.2
- new net: D5.2 (A), S5.2
- new net: D17.2 (A), S17.2
- new net: D14.2 (A), S14.2
- new net: D11.2 (A), S11.2
- new net BAT+: PSW1.3 (C), PSW2.1 (A), U1.24 (BATIN/P0.04)
- new net ENC_A: SW22.A, U1.16 (P1.13)
- new net ENC_B: SW22.B, U1.15 (P1.11)
- new net GND: J1.2 (Pin_2), RSW1.2, RSW2.1, SW22.C, U1.23 (GND), U1.3 (GND), U1.4 (GND)
- new net R1: D1.1 (K), D10.1 (K), D13.1 (K), D16.1 (K), D4.1 (K), D7.1 (K), U1.11 (P1.04)
- new net R2: D11.1 (K), D14.1 (K), D17.1 (K), D2.1 (K), D5.1 (K), D8.1 (K), U1.13 (NFC1/P0.09)
- new net R3: D12.1 (K), D15.1 (K), D18.1 (K), D3.1 (K), D6.1 (K), D9.1 (K), U1.7 (P0.22)
- new net R4: D19.1 (K), D20.1 (K), D21.1 (K), D22.1 (K), U1.14 (NFC2/P0.10)
- new net VBAT: J1.1 (Pin_1), PSW1.2 (B), PSW2.2 (B)
- no-connect marks 5 -> 12
Other:
- note added: "HOOKAH-WL"
- note added: "MCU"
- note added: "MOUNTING HOLES"
- note removed: "L E F T"
- note removed: "M I C R O C O N T R O L L E R"
- note removed: "T O T E M"
- title: TOTEM split keyboard -> Hookah Wireless Split
- moved on the sheet: RSW1, S1, S10, S11, S12, S13, S14, S15, S16, S17, S18, S19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
