File: PCB/hookah-wl/hookah/hookah.kicad_pcb (KiCad board)
At the start: 2 copper layers, 146.6 x 102.4 mm, 72 parts, among them J1 Conn_01x02_Socket, J2 Conn_01x12_Socket, J4 Conn_01x04, J5 Conn_01x04, J6 Conn_01x12_Socket, SW1 RotaryEncoder_Switch, SW22 RotaryEncoder_Switch, U1 nice_nano

Commit message: Hookah WL final
Parts:
- removed JP1, JP2, JP3, JP4: ~, hookah-wl:Reversible-Jumper
- removed Nice!View1: ~, hookah-wl:Nice!View
- removed the RSW1 at (178.4, 77.9)
- removed the RSW2 at (178.4, 77.9)
- R2: moved to B.Cu
- moved RSW1 25.1 mm to (178.0, 76.7)
- moved RSW2 25.1 mm to (178.0, 76.7)
- moved R2 15.7 mm to (101.4, 104.7)
- moved J1 0.93 mm to (191.1, 76.2)
Connections:
- U1 pad 10: CS -> unconnected-(U1-P0.11-Pad10)
- U1 pad 12: SCK -> unconnected-(U1-P1.06-Pad12)_1
- U1 pad 9: MOSI -> unconnected-(U1-P1.00-Pad9)_1
Routing:
- net MOSI: track 28.7 -> 0.00 mm, vias 5 -> 0
- net CS: track 19.9 -> 0.00 mm, vias 3 -> 0
- net SCK: track 18.1 -> 0.00 mm, vias 2 -> 0
- net VCC: track 177.9 -> 165.6 mm
- net DISP_CS/MOSI: track 7.08 -> 0.00 mm
- net DISP_MOSI/CS: track 6.68 -> 0.00 mm
- net DISP_SCK/GND: track 6.34 -> 0.00 mm
- net DISP_GND/SCK: track 6.19 -> 0.00 mm
- net TP_DATA: track 157.2 -> 159.7 mm, vias 4 -> 3
- net R1: track 140.6 -> 138.4 mm
- net RESET: track 59.3 -> 61.1 mm, vias 3 -> 5
- net R4: track 137.5 -> 135.8 mm
- net VBAT: track 50.1 -> 49.1 mm
- net Net-(J4-Pin_3): track 43.0 -> 42.2 mm
- net /ENC_A: track 92.0 -> 91.5 mm
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