File: PCB/hookah-wl/hookah/hookah.kicad_sch (KiCad schematic)
At the start: 70 parts, among them J1 Conn_01x02_Socket, J2 Conn_01x12_Socket, J4 Conn_01x04, J5 Conn_01x04, J6 Conn_01x12_Socket, SW1 RotaryEncoder_Switch, SW22 RotaryEncoder_Switch, U1 nice_nano

Commit message: Hookah WL final
Parts:
- removed JP1, JP2, JP3, JP4: ~, hookah-wl:Reversible-Jumper, symbol hookah-wl:Reversible_Jumper
- removed Nice!View1: ~, hookah-wl:Nice!View, symbol hookah-wl:Nice!View
Connections:
- net CS: no longer names the net of U1.10 (P0.11)
- net MOSI: no longer names the net of U1.9 (P1.00)
- net SCK: no longer names the net of U1.12 (P1.06)
- no-connect marks 20 -> 23
